File: PCB/ESPHomeCover/motor_driver.kicad_sch (KiCad schematic)
At the start: 18 parts, among them IC2 DRV8425PWPR, K1 G6S-2(F)-Y_DC24, Q1 MMBF170, X5 Motor, X6 Brake

Commit message: Add Board
Parts:
- added J7: ~, Connector_PinHeader_2.54mm:PinHeader_1x03_P2.54mm_Vertical, symbol Connector_Generic:Conn_01x03
- C10: value 0.022uF X7R 36V -> 0.022uF X7R 50V; footprint (none) -> Capacitor_SMD:C_0805_2012Metric; LCSC (none) -> C107147
- C11: footprint (none) -> Capacitor_SMD:C_0805_2012Metric; LCSC (none) -> C3869051
- C12: value 100uF 36V -> 100uF 35V; footprint (none) -> Capacitor_SMD:CP_Elec_6.3x7.7; LCSC (none) -> C72478
- C7: footprint (none) -> Capacitor_SMD:C_0805_2012Metric; LCSC (none) -> C113853
- C8, C9: value 0.01uF 36V -> 0.01uF 35V; footprint (none) -> Capacitor_SMD:C_0402_1005Metric; LCSC (none) -> C1518210
- D1: footprint Diode_SMD:D_SMA -> Diode_THT:D_DO-41_SOD81_P10.16mm_Horizontal
- J5: renamed from X5; footprint (none) -> Connector_JST:JST_XH_B4B-XH-A_1x04_P2.50mm_Vertical
- J6: renamed from X6; footprint (none) -> Connector_JST:JST_XH_B3B-XH-A_1x03_P2.50mm_Vertical; symbol Connector_Generic:Conn_01x02 -> Connector_Generic:Conn_01x03
- JP2, JP3: footprint (none) -> Connector_PinHeader_2.54mm:PinHeader_1x03_P2.54mm_Vertical_SMD_Pin1Left; LCSC (none) -> C780061
- K1: footprint SamacSys_Parts:G6S2FYDC24 -> Own_Lib:G6S2(F)YDC24; symbol SamacSys_Parts:G6S-2F-Y_DC24 -> own lib:G6S-2(F)-Y_DC24; LCSC C1525796 -> C1525293; LCSC Part (none) -> C1525796
- R4: footprint (none) -> Resistor_SMD:R_0805_2012Metric; LCSC (none) -> C149504
- R5: footprint (none) -> Resistor_SMD:R_0805_2012Metric; LCSC (none) -> C4328
- R6: footprint (none) -> Resistor_SMD:R_0805_2012Metric; LCSC (none) -> C17455
- R7: footprint (none) -> Resistor_SMD:R_0805_2012Metric; LCSC (none) -> C17414
- renumbered IC2 to U2
Connections:
- net DVDD is gone; now on net +3V3: JP2.1 (A), JP3.1 (A)
- net at J6.1 (Pin_1): now also K1.3 (NC_1); no longer K1.4 (COM_1)
- net at J6.2 (Pin_2): now also K1.4 (COM_1); no longer K1.5 (NO_1)
- net at K1.10 (NC_2): now also J7.1 (Pin_1)
- net at K1.8 (NO_2): now also J7.3 (Pin_3)
- net at K1.9 (COM_2): now also J7.2 (Pin_2)
- new net: J6.3 (Pin_3), K1.5 (NO_1)
- no-connect marks 4 -> 0
Other:
- moved on the sheet: C12, R4, R5, R6

Commit message: small changes
change all Caps to 0603,
add bom
Parts:
- C10: footprint Capacitor_SMD:C_0805_2012Metric -> Capacitor_SMD:C_0603_1608Metric; LCSC C107147 -> C77571
- C11: footprint Capacitor_SMD:C_0805_2012Metric -> Capacitor_SMD:C_0603_1608Metric; LCSC C3869051 -> C309479
- C7: footprint Capacitor_SMD:C_0805_2012Metric -> Capacitor_SMD:C_0603_1608Metric; LCSC C113853 -> (none)
- C8, C9: footprint Capacitor_SMD:C_0402_1005Metric -> Capacitor_SMD:C_0603_1608Metric; LCSC C1518210 -> (none)
Other:
- company: (none) -> Tim
Changed lines of the file:
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@@
 	(title_block
 		(title "ESPHome Cover PCB")
-		(date "2024-05-08")
-		(rev "1")
+		(date "2024-05-12")
+		(rev "2")
+		(company "Tim")
 	)
 	(junction
@@
 			)
 		)
-		(property "Footprint" "Capacitor_SMD:C_0805_2012Metric"
+		(property "Footprint" "Capacitor_SMD:C_0603_1608Metric"
 			(at 124.1552 72.39 0)
 			(effects
@@
 			)
 		)
-		(property "LCSC" "C113853"
+		(property "LCSC" ""
+			(at 123.19 68.58 0)
+			(effects
+				(font
+					(size 1.27 1.27)
+				)
+				(hide yes)
+			)
+		)
+		(property "Mouser" ""
 			(at 123.19 68.58 0)
 			(effects
@@
 			)
 		)
+		(property "Mouser" ""
+			(at 102.87 82.55 0)
+			(effects
+				(font
+					(size 1.27 1.27)
+				)
+				(hide yes)
+			)
+		)
 		(pin "2"
 		)
@@
 			)
 		)
-		(property "Footprint" "Capacitor_SMD:C_0805_2012Metric"
+		(property "Footprint" "Capacitor_SMD:C_0603_1608Metric"
 			(at 168.6052 110.49 0)
 			(effects
@@
 			)
 		)
-		(property "LCSC" "C3869051"
+		(property "LCSC" "C309479"
+			(at 167.64 106.68 0)
+			(effects
+				(font
+					(size 1.27 1.27)
+				)
+				(hide yes)
+			)
+		)
+		(property "Mouser" ""
 			(at 167.64 106.68 0)
 			(effects
@@
 			)
 		)
+		(property "Mouser" ""
+			(at 231.14 41.91 0)
+			(effects
+				(font
+					(size 1.27 1.27)
+				)
+				(hide yes)
+			)
+		)
 		(pin "2"
 		)
@@
 			)
 		)
+		(property "Mouser" ""
+			(at 129.54 69.85 0)
+			(effects
+				(font
+					(size 1.27 1.27)
+				)
+				(hide yes)
+			)
+		)
 		(pin "21"
 		)
@@
 			)
 		)
+		(property "Mouser" ""
+			(at 257.81 41.91 0)
+			(effects
+				(font
+					(size 1.27 1.27)
+				)
+				(hide yes)
+			)
+		)
 		(pin "2"
 		)
@@
 			)
 		)
+		(property "Mouser" ""
+			(at 193.04 81.28 0)
+			(effects
+				(font
+					(size 1.27 1.27)
+				)
+				(hide yes)
+			)
+		)
 		(pin "1"
 		)
@@
 			)
 		)
+		(property "Mouser" ""
+			(at 118.11 119.38 0)
+			(effects
+				(font
+					(size 1.27 1.27)
+				)
+				(hide yes)
+			)
+		)
 		(pin "1"
 		)
@@
 			)
 		)
+		(property "Mouser" ""
+			(at 35.56 173.99 0)
+			(effects
+				(font
+					(size 1.27 1.27)
+				)
+				(hide yes)
+			)
+		)
 		(pin "1"
 		)
@@
 			)
 		)
+		(property "Mouser" ""
+			(at 74.93 156.21 0)
+			(effects
+				(font
+					(size 1.27 1.27)
+				)
+				(hide yes)
+			)
+		)
 		(pin "2"
 		)
@@
 			)
 		)
-		(property "Footprint" "Capacitor_SMD:C_0402_1005Metric"
+		(property "Footprint" "Capacitor_SMD:C_0603_1608Metric"
 			(at 113.03 71.4248 0)
 			(effects
@@
 			)
 		)
-		(property "LCSC" "C1518210"
+		(property "LCSC" ""
+			(at 109.22 72.39 0)
+			(effects
+				(font
+					(size 1.27 1.27)
+				)
+				(hide yes)
+			)
+		)
+		(property "Mouser" ""
 			(at 109.22 72.39 0)
 			(effects
@@
 			)
 		)
+		(property "Mouser" ""
+			(at 107.95 160.02 0)
+			(effects
+				(font
+					(size 1.27 1.27)
+				)
+				(hide yes)
+			)
+		)
 		(pin "1"
 		)
@@
 			)
 		)
+		(property "Mouser" ""
+			(at 196.85 69.85 0)
+			(effects
+				(font
+					(size 1.27 1.27)
+				)
+				(hide yes)
+			)
+		)
 		(pin "2"
 		)
@@
 			)
 		)
+		(property "Mouser" ""
+			(at 196.85 81.28 0)
+			(effects
+				(font
+					(size 1.27 1.27)
+				)
+				(hide yes)
+			)
+		)
 		(pin "2"
 		)
@@
 			)
 		)
-		(property "Footprint" "Capacitor_SMD:C_0805_2012Metric"
+		(property "Footprint" "Capacitor_SMD:C_0603_1608Metric"
 			(at 173.6852 72.39 0)
 			(effects
@@
 			)
 		)
-		(property "LCSC" "C107147"
+		(property "LCSC" "C77571"
+			(at 172.72 68.58 0)
+			(effects
+				(font
+					(size 1.27 1.27)
+				)
+				(hide yes)
+			)
+		)
+		(property "Mouser" ""
 			(at 172.72 68.58 0)
 			(effects
@@
 			)
 		)
+		(property "Mouser" ""
+			(at 85.09 186.69 0)
+			(effects
+				(font
+					(size 1.27 1.27)
+				)
+				(hide yes)
+			)
+		)
 		(pin "1"
 		)
@@
 			)
 		)
+		(property "Mouser" ""
+			(at 100.33 166.37 0)
+			(effects
+				(font
+					(size 1.27 1.27)
+				)
+				(hide yes)
+			)
+		)
 		(pin "3"
 		)
@@
 			)
 		)
+		(property "Mouser" ""
+			(at 59.69 168.91 0)
+			(effects
+				(font
+					(size 1.27 1.27)
+				)
+				(hide yes)
+			)
+		)
 		(pin "12"
 		)
@@
 			)
 		)
-		(property "Footprint" "Capacitor_SMD:C_0402_1005Metric"
+		(property "Footprint" "Capacitor_SMD:C_0603_1608Metric"
 			(at 113.03 99.3648 0)
 			(effects
@@
 			)
 		)
-		(property "LCSC" "C1518210"
+		(property "LCSC" ""
+			(at 109.22 100.33 0)
+			(effects
+				(font
+					(size 1.27 1.27)
+				)
+				(hide yes)
+			)
+		)
+		(property "Mouser" ""
 			(at 109.22 100.33 0)
 			(effects

Commit message: update PCB
Parts:
- C10: Mouser Part Number (none) -> 581-06035C223KAT4A
- C11: Mouser Part Number (none) -> 581-06035C105KAT2A
- C12: Mouser Part Number (none) -> 667-EEH-ZK1V101XP
- C7: Mouser Part Number (none) -> 80-C0603C224K4R
- C8, C9: Mouser Part Number (none) -> 810-C1608C0G1V153JAC
- D1: Mouser Part Number (none) -> 637-1N4001
- Q1: Mouser Part Number (none) -> 512-MMBF170
- R4: Mouser Part Number (none) -> 71-CRCW0805100KJNECC
- R5: Mouser Part Number (none) -> 71-CRCW080520K0FKEAH
- R6: Mouser Part Number (none) -> 71-CRCW080513K0JNEA
- R7: Mouser Part Number (none) -> 667-ERA-6AEB103V
- renumbered J5 to J4, J6 to J5, J7 to J6, JP2 to JP1, JP3 to JP2, U2 to U1
Changed lines of the file:
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@@
 		(title "ESPHome Cover PCB")
 		(date "2024-05-12")
-		(rev "2")
+		(rev "1")
 		(company "Tim")
 	)
@@
 	)
 	(junction
+		(at 114.3 72.39)
+		(diameter 0)
+		(color 0 0 0 0)
+	)
+	(junction
 		(at 92.71 168.91)
 		(diameter 0)
@@
 	(wire
 		(pts
-			(xy 114.3 106.68) (xy 114.3 100.33)
+			(xy 114.3 109.22) (xy 114.3 100.33)
 		)
 		(stroke
@@
 	(wire
 		(pts
+			(xy 114.3 63.5) (xy 114.3 72.39)
+		)
+		(stroke
+			(width 0)
+			(type default)
+		)
+	)
+	(wire
+		(pts
 			(xy 90.17 176.53) (xy 92.71 176.53)
 		)
@@
 	(wire
 		(pts
+			(xy 114.3 72.39) (xy 123.19 72.39)
+		)
+		(stroke
+			(width 0)
+			(type default)
+		)
+	)
+	(wire
+		(pts
 			(xy 50.8 168.91) (xy 57.15 168.91)
 		)
@@
 	(wire
 		(pts
+			(xy 101.6 63.5) (xy 114.3 63.5)
+		)
+		(stroke
+			(width 0)
+			(type default)
+		)
+	)
+	(wire
+		(pts
 			(xy 100.33 152.4) (xy 100.33 160.02)
 		)
@@
 	(wire
 		(pts
-			(xy 101.6 106.68) (xy 114.3 106.68)
+			(xy 101.6 109.22) (xy 114.3 109.22)
 		)
 		(stroke
@@
 	(wire
 		(pts
-			(xy 113.03 72.39) (xy 123.19 72.39)
+			(xy 113.03 72.39) (xy 114.3 72.39)
 		)
 		(stroke
@@
 	)
 	(label "+24V"
-		(at 101.6 106.68 0)
+		(at 101.6 109.22 0)
 		(fields_autoplaced yes)
 		(effects
@@
 	)
 	(label "+24V"
-		(at 113.03 72.39 0)
+		(at 101.6 63.5 0)
 		(fields_autoplaced yes)
 		(effects
@@
 			)
 		)
+		(property "Mouser Part Number" "80-C0603C224K4R"
+			(at 123.19 68.58 0)
+			(effects
+				(font
+					(size 1.27 1.27)
+				)
+				(hide yes)
+			)
+		)
 		(pin "1"
 		)
@@
 		(on_board yes)
 		(dnp no)
-		(property "Reference" "J5"
+		(property "Reference" "J4"
 			(at 98.298 81.788 0)
 			(effects
@@
 			(project "ESPHomeCover"
 				(path "/457ec9a0-69c6-4fbc-b0c1-e7e1db8d25f0/ba731c15-d691-4401-90d0-2f66281d5c9f"
-					(reference "J5")
+					(reference "J4")
 					(unit 1)
 				)
@@
 			)
 		)
+		(property "Mouser Part Number" "581-06035C105KAT2A"
+			(at 167.64 106.68 0)
+			(effects
+				(font
+					(size 1.27 1.27)
+				)
+				(hide yes)
+			)
+		)
 		(pin "1"
 		)
@@
 		(dnp no)
 		(fields_autoplaced yes)
-		(property "Reference" "JP3"
+		(property "Reference" "JP2"
 			(at 233.68 40.6399 90)
 			(effects
@@
 			(project "ESPHomeCover"
 				(path "/457ec9a0-69c6-4fbc-b0c1-e7e1db8d25f0/ba731c15-d691-4401-90d0-2f66281d5c9f"
-					(reference "JP3")
+					(reference "JP2")
 					(unit 1)
 				)
@@
 		(dnp no)
 		(fields_autoplaced yes)
-		(property "Reference" "U2"
+		(property "Reference" "U1"
 			(at 147.32 62.23 0)
 			(effects
@@
 			(project "ESPHomeCover"
 				(path "/457ec9a0-69c6-4fbc-b0c1-e7e1db8d25f0/ba731c15-d691-4401-90d0-2f66281d5c9f"
-					(reference "U2")
+					(reference "U1")
 					(unit 1)
 				)
@@
 		(dnp no)
 		(fields_autoplaced yes)
-		(property "Reference" "JP2"
+		(property "Reference" "JP1"
 			(at 260.35 40.6399 90)
 			(effects
@@
 			(project "ESPHomeCover"
 				(path "/457ec9a0-69c6-4fbc-b0c1-e7e1db8d25f0/ba731c15-d691-4401-90d0-2f66281d5c9f"
-					(reference "JP2")
+					(reference "JP1")
 					(unit 1)
 				)
@@
 			)
 		)
+		(property "Mouser Part Number" "71-CRCW0805100KJNECC"
+			(at 193.04 81.28 0)
+			(effects
+				(font
+					(size 1.27 1.27)
+				)
+				(hide yes)
+			)
+		)
 		(pin "1"
 		)
@@
 			)
 		)
+		(property "Mouser Part Number" "667-EEH-ZK1V101XP"
+			(at 118.11 119.38 0)
+			(effects
+				(font
+					(size 1.27 1.27)
+				)
+				(hide yes)
+			)
+		)
 		(pin "1"
 		)
@@
 		(on_board yes)
 		(dnp no)
-		(property "Reference" "J6"
+		(property "Reference" "J5"
 			(at 30.734 173.736 0)
 			(effects
@@
 			(project "ESPHomeCover"
 				(path "/457ec9a0-69c6-4fbc-b0c1-e7e1db8d25f0/ba731c15-d691-4401-90d0-2f66281d5c9f"
-					(reference "J6")
+					(reference "J5")
 					(unit 1)
 				)
@@
 			)
 		)
+		(property "Mouser Part Number" "637-1N4001"
+			(at 74.93 156.21 0)
+			(effects
+				(font
+					(size 1.27 1.27)
+				)
+				(hide yes)
+			)
+		)
 		(pin "2"
 		)
@@
 		)
 		(property "Value" "0.01uF 35V"
-			(at 109.22 68.58 90)
+			(at 107.95 68.58 90)
 			(effects
 				(font
@@
 			)
 		)
+		(property "Mouser Part Number" "810-C1608C0G1V153JAC"
+			(at 109.22 72.39 0)
+			(effects
+				(font
+					(size 1.27 1.27)
+				)
+				(hide yes)
+			)
+		)
 		(pin "2"
 		)
@@
 			)
 		)
+		(property "Mouser Part Number" "667-ERA-6AEB103V"
+			(at 107.95 160.02 0)
+			(effects
+				(font
+					(size 1.27 1.27)
+				)
+				(hide yes)
+			)
+		)
 		(pin "1"
 		)
@@
 			)
 		)
+		(property "Mouser Part Number" "71-CRCW080513K0JNEA"
+			(at 196.85 69.85 0)
+			(effects
+				(font
+					(size 1.27 1.27)
+				)
+				(hide yes)
+			)
+		)
 		(pin "2"
 		)
@@
 			)
 		)
+		(property "Mouser Part Number" "71-CRCW080520K0FKEAH"
+			(at 196.85 81.28 0)
+			(effects
+				(font
+					(size 1.27 1.27)
+				)
+				(hide yes)
+			)
+		)
 		(pin "2"
 		)
@@
 			)
 		)
+		(property "Mouser Part Number" "581-06035C223KAT4A"
+			(at 172.72 68.58 0)
+			(effects
+				(font
+					(size 1.27 1.27)
+				)
+				(hide yes)
+			)
+		)
 		(pin "1"
 		)
@@
 		(on_board yes)
 		(dnp yes)
-		(property "Reference" "J7"
+		(property "Reference" "J6"
 			(at 81.534 186.944 0)
 			(effects
@@
 			(project "ESPHomeCover"
 				(path "/457ec9a0-69c6-4fbc-b0c1-e7e1db8d25f0/ba731c15-d691-4401-90d0-2f66281d5c9f"
-					(reference "J7")
+					(reference "J6")
 					(unit 1)
 				)
@@
 			)
 		)
+		(property "Mouser Part Number" "512-MMBF170"
+			(at 100.33 166.37 0)
+			(effects
+				(font
+					(size 1.27 1.27)
+				)
+				(hide yes)
+			)
+		)
 		(pin "3"
 		)
@@
 			(at 109.22 100.33 0)
 			(effects
+				(font
+					(size 1.27 1.27)
+				)
+				(hide yes)
+			)
+		)
+		(property "Mouser Part Number" "810-C1608C0G1V153JAC"
+			(at 109.22 100.33 0)
+			(effects
